File: hardware/Lentes EKOparty-2024/Lentes EKOparty-2024.kicad_sch (KiCad schematic)
At the start: 1 part, among them J2 Conn_02x03_Odd_Even

Commit message: feat(Hw):Added_Lentes_BoM
Parts:
- J2: #LCSC C124390 -> C706893
Changed lines of the file:
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@@
 			)
 		)
-		(property "#LCSC" "C124390"
+		(property "#LCSC" "C706893"
 			(at 39.116 37.592 0)
 			(effects
